File: RAT_pedal.kicad_pcb (KiCad board)
At the start: 2 copper layers, 42 x 42 mm, 41 parts, among them J1 GNDREF_PIN, J2 INPUT_PIN, J3 OUTPUT_PIN, J4 LED+, J5 POWER_IN, Q1 2N5458, U1 LM308

Commit message: Updates yo
Parts:
- moved C11 13.8 mm to (144.5, 71.3)
- moved D1 8.89 mm to (140.1, 57.1), turned to 180 degrees
- moved TP1 4.86 mm to (136.5, 63.4)
- moved C13 4.78 mm to (144.4, 62.8), turned to 180 degrees
- moved R12 4.24 mm to (145.6, 67.3)
- moved D2 2.64 mm to (132.4, 59.6), turned to 0 degrees
- moved C7 2.00 mm to (135.3, 71.5), turned to 180 degrees
- moved C6 1.99 mm to (118.1, 57.7), turned to 180 degrees
- moved C5 1.93 mm to (141.6, 90.3), turned to 180 degrees
- moved R11 1.54 mm to (140.6, 75.1)
- moved C10 0.41 mm to (150.7, 59.0), turned to 180 degrees
- moved J1 0.18 mm to (147.9, 92.9)
- moved J2 0.14 mm to (145.6, 92.9)
Routing:
- net VB: track 16.1 -> 22.8 mm
- net Net-(C7-Pad2): track 6.42 -> 4.54 mm
- net Net-(C10-Pad2): track 6.36 -> 4.55 mm
- net Net-(C5-Pad1): track 15.3 -> 16.9 mm
- net Net-(D1-A): track 13.8 -> 14.8 mm
- net Net-(C6-Pad1): track 17.9 -> 18.8 mm
- net Net-(C4-Pad2): track 25.3 -> 26.1 mm
- net +9V: track 91.3 -> 90.5 mm
