File: RAT_pedal.kicad_sch (KiCad schematic)
At the start: 41 parts, among them J1 GNDREF_PIN, J2 INPUT_PIN, J3 OUTPUT_PIN, J4 LED+, J5 POWER_IN, Q1 2N5458, U1 LM308

Commit message: Updates yo
Other:
- moved on the sheet: C10, C2, C3, R6, R9
